File: SpeedJeck.kicad_sch (KiCad schematic)
At the start: 18 parts, among them J2 USB_A, SW1 SW_Push, SW2 SW_Push, SW3 SW_Push, SW4 SW_Push, SW5 SW_Push, SW6 SW_Push, U2 Adafruit SSD1306, U3 AMS1117-3.3

Commit message: [schEMATIC] [VERSION CODE 1v] [Ref 2], [PCB] [version code 1] [rev 1] [13.11.2025] [Final SPEEDJECK 1v]
Parts:
- removed U3: AMS1117-3.3, Package_TO_SOT_SMD:SOT-223, symbol Arduino_modules:AMS1117
- added U3: AMS1117-3.3, Package_TO_SOT_SMD:SOT-223-3_TabPin2, symbol Regulator_Linear:AMS1117-3.3
- U2: value Adafruit SSD1306 -> Adafruit SSD1306 1.3 inch; footprint (none) -> SC:LCD_OLED_128X64_1.3_I2C
- renumbered J2 to J1, SW5 to SW2, SW2 to SW3, SW3 to SW5
Connections:
- net +3.3V: now also U3.2 (VO)
- net D10: now also SW3.1; no longer SW4.1
- net D11: now also SW2.1; no longer SW3.1
- net D12: now also SW1.1; no longer SW2.1
- net D8: now also SW5.1; no longer SW6.1
- net D9: now also SW4.1; no longer SW5.1
- net GND: now also U3.1 (GND)
- net D7: now reaches A1.10 (D7)
- net D7: now also SW6.1
- net at J1.1 (VBUS): now also U3.3 (VI)
- net D13: no longer names the net of A1.16 (D13)
- net D13: no longer SW1.1
