File: SpeedJeck.kicad_sch (KiCad schematic)
At the start: 18 parts, among them J1 USB_A, SW1 SW_Push, SW2 SW_Push, SW3 SW_Push, SW4 SW_Push, SW5 SW_Push, SW6 SW_Push, U2 Adafruit SSD1306 1.3 inch, U3 AMS1117-3.3

Commit message: [Replacement a component 2k2] [MANUFACTURE] [LCSC components] [JLCPCB] [version code 1] [01.12.2025] [SPEEDJECK 1v]
Parts:
- R1: LCSC C4146660 -> C25879
Changed lines of the file:
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@@
 			)
 		)
-		(property "LCSC" "C4146660"
+		(property "LCSC" "C25879"
 			(at 52.07 44.45 0)
 			(effects
