File: SpeedJeck.kicad_pcb_BAc2025.11.28[LCSC_PCB].kicad_pcb (KiCad board)
At the start: 2 copper layers, 94 x 58 mm, 23 parts, among them U2 Adafruit SSD1306 1.3 inch, U3 AMS1117-3.3

Commit message: [MANUFACTURE] [LCSC components] [JLCPCB] [version code 1] [28.11.2025] [SPEEDJECK 1v]
Parts:
- BZ1: footprint SC:BUZ-TH_BD12.0-P7.60-D0.6-FD -> Buzzer_Beeper:MagneticBuzzer_ProSignal_ABT-410-RC
- R7, R8: footprint Resistor_SMD:R_0603_1608Metric -> Resistor_SMD:R_0402_1005Metric
- moved BZ1 4.22 mm to (149.0, 44.0)
- moved R1 1.22 mm to (135.5, 82.0)
- moved R7 0.70 mm to (135.5, 85.0)
- moved R8 0.63 mm to (135.5, 88.0)
Routing:
- net GND: track 19.9 -> 27.5 mm
- net D5: track 59.4 -> 58.2 mm
- net D4: track 58.2 -> 57.4 mm
- net /Data+: track 24.8 -> 25.4 mm
- net /Data-: track 26.6 -> 27.1 mm
